File: hardware/main.brd (EAGLE design)
At the start: 65 x 56.5 mm, 58 parts

Commit message: Hardware revision 2, as ordered.
Parts:
- removed R9: 100k, rcl:R0603
- removed SERVO1, SERVO2, SERVO3, SERVO4: HDR_1X3, bleHAT:HDR_1X3
- removed U$8: TXB0104, bleHAT:TSSOP14
- added 3V3_PI, CS0, CS1, CS2, CS3, CS4, CS5, R16, R17, R8, R_DRDY, R_INT1, R_INT2, R_SCL, R_SDA: (no value), rcl:R0603
- added C18, C19, C20, C21, C22, C8: (no value), resistor:C0603
- added JP6: (no value), bleHAT:1X06
- added PWM1, PWM2, PWM3, PWM4: HDR_1X3, bleHAT:HDR_1X3
- added R22, R23, R24, R25, R30, R31: (no value), resistor:R1206
- added U$5, U$7: DRV8838, bleHAT:WSON-8-PAD
- JP2: device bleHAT:1X07 -> bleHAT:1X05
- JP3: device bleHAT:1X05 -> bleHAT:1X06
- JP4: device bleHAT:1X03 -> bleHAT:1X02
- JP5: device pinhead:1X01 -> bleHAT:1X02
- moved WS2 56.9 mm to (63.1, 43.7), turned to 270 degrees
- moved WS4 52.2 mm to (53.2, 34.4)
- moved U$12 48.9 mm to (8.26, 41.9), turned to 270 degrees
- moved C14 46.8 mm to (11.4, 4.32), turned to 180 degrees
- moved 3V3_LDO 42.6 mm to (11.4, 8.00), turned to 0 degrees
- moved C13 42.5 mm to (11.6, 11.6), turned to 180 degrees
- moved C11 39.1 mm to (21.3, 48.8), turned to 0 degrees
- moved R15 37.7 mm to (12.4, 43.3), flipped to the bottom, turned to 270 degrees
- moved POWER 37.5 mm to (6.10, 43.1), turned to 90 degrees
- moved R6 37.4 mm to (50.2, 35.6), turned to 0 degrees
- moved R7 37.0 mm to (50.2, 33.0), turned to 0 degrees
- moved PCT2075 36.8 mm to (22.7, 42.9), flipped to the bottom, turned to 90 degrees
- moved U$2 36.2 mm to (4.57, 11.0), turned to 270 degrees
- moved R14 35.6 mm to (16.4, 43.6), flipped to the bottom, turned to 270 degrees
- moved R3 35.3 mm to (49.0, 41.9), turned to 0 degrees
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Connections:
- removed net N$36: R9.1, U$8.8
- removed net PDWN_N: BLE112A.15, JP3.1, U$3.4
- removed net PWM1_5V0: SERVO4.2, U$8.10
- removed net PWM2_5V0: SERVO3.2, U$8.11
- removed net PWM3_5V0: SERVO2.2, U$8.12
- removed net PWM4_5V0: SERVO1.2, U$8.13
- new net 3V3_PI: 3V3_PI.1, C11.2, PCT2075.8, R14.2, R15.2, U$4.1, U$4.14, U$4.7
- new net 3V3_PI_BYP: 3V3_PI.2, JP1.1
- new net GPIO17_PI: JP1.11, R_INT2.2
- new net GPIO18_PI: JP1.12, R_DRDY.1
- new net GPIO4_PI: JP1.7, R_INT1.2
- new net I2C_SCL_PI: JP1.5, R_SCL.2
- new net I2C_SDA_PI: JP1.3, R_SDA.2
- new net N$12: JP4.1, U$5.3
- new net N$13: CS2.2, PWM2.3, R22.1
- new net N$14: CS3.1, PWM1.3, R23.1
- new net N$15: CS0.2, PWM4.3, R25.2
- new net N$16: CS1.1, PWM3.3, R24.2
- new net N$21: JP4.2, U$5.2
- new net N$22: JP5.1, U$7.3
- new net N$23: JP5.2, U$7.2
- new net N$26: CS4.1, R30.2, U$5.4
- new net N$27: CS5.1, R31.2, U$7.4
- new net P1_0: BLE112A.18, JP3.4, R17.1
- new net P2_0: BLE112A.6, JP2.3
- new net SLEEP_N: BLE112A.15, JP3.1, U$3.4, U$5.7, U$7.7
- new net TMR3_PWM0: BLE112A.8, JP2.5, U$7.5
- new net TMR3_PWM1: BLE112A.7, JP2.4, U$5.5
- new net USB+: BLE112A.11, R17.2, R8.2
- new net USB-: BLE112A.12, R16.2
- net 3V3: now also U$5.8, U$7.8; no longer C11.2, PCT2075.8, R14.2, R15.2, R9.2, U$4.1, U$4.14, U$4.7, U$8.1
- net 5V0: now also C18.2, C19.2, C20.2, C21.2, C22.2, C8.2, PWM1.2, PWM2.2, PWM3.2, PWM4.2, U$5.1, U$7.1; no longer SERVO1.1, SERVO2.1, SERVO3.1, SERVO4.1, U$8.14
- net AIN0: now also CS4.2
- net AIN1: now also CS5.2
- net AIN4: now also CS3.2
- net AIN5: now also CS2.1
- net AIN6: now also CS0.1
- net AIN7: now also CS1.2
- net ANALOG0: now also JP6.1; no longer JP2.7
- net ANALOG1: now also JP6.2; no longer JP2.6
- net DC: now also JP2.1, U$7.6
- net DD: now also JP2.2, U$5.6
- net DRDY_N: now also R_DRDY.2; no longer BLE112A.16, JP2.1
- net GND: now also C18.1, C19.1, C20.1, C21.1, C22.1, C8.1, R22.2, R23.2, R24.1, R25.1, R30.1, R31.1; no longer SERVO1.3, SERVO2.3, SERVO3.3, SERVO4.3, U$8.7
- net INT1: now also R_INT1.1; no longer JP5.1
- net INT2: now also R_INT2.1; no longer BLE112A.6, JP4.1
- net N$3: now also R8.1; no longer BLE112A.11
- net N$4: now also R16.1; no longer BLE112A.12
- net PWM1: now also BLE112A.16, PWM1.1; no longer BLE112A.17, U$8.5
- net PWM2: now also BLE112A.17, PWM2.1; no longer BLE112A.18, U$8.4
- net PWM3: now also JP3.5, PWM3.1; no longer JP3.4, U$8.3
- net PWM4: now also JP3.6, PWM4.1; no longer JP3.5, U$8.2
- net SCL: now also R_SCL.1; no longer BLE112A.7, JP4.2
- net SDA: now also R_SDA.1; no longer BLE112A.8, JP4.3
- net SPI_CLK: now also JP6.4; no longer JP2.4
- net SPI_MISO: now also JP6.6; no longer JP2.2
- net SPI_MOSI: now also JP6.5; no longer JP2.3
- net SPI_SS: now also JP6.3; no longer JP2.5
Routing:
- net PWM2_5V0: track 57.3 -> 0.00 mm, vias 2 -> 0
- net SLEEP_N: track 0.00 -> 50.2 mm, vias 0 -> 3
- net 3V3_PI: track 0.00 -> 48.5 mm, vias 0 -> 3
- net PWM2: track 9.79 -> 56.7 mm, vias 0 -> 4
- net PWM1_5V0: track 46.3 -> 0.00 mm, vias 2 -> 0
- net DC: track 31.0 -> 74.2 mm, vias 2 -> 1
- net PWM3: track 10.3 -> 52.7 mm, vias 0 -> 2
- net 3V3: track 208.6 -> 169.4 mm, vias 12 -> 11
- net TMR3_PWM0: track 0.00 -> 38.4 mm, vias 0 -> 1
- net PWM3_5V0: track 37.1 -> 0.00 mm, vias 3 -> 0
- net PWM1: track 11.1 -> 47.3 mm, vias 0 -> 1
- net DD: track 26.5 -> 62.6 mm, vias 2 -> 1
- net PWM4: track 13.2 -> 45.9 mm, vias 0 -> 2
- net TMR3_PWM1: track 0.00 -> 31.3 mm, vias 0 -> 1
- net N$5: track 0.00 -> 30.7 mm, vias 0 -> 2
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- added copper zone on layer 1, net 3V3
- added copper zone on layer 1, net 5V0
- added copper zone on layer 1, net N$26
- added copper zone on layer 1, net N$27
- added copper zone on layer 16, net N$5
- added copper zone on layer 16, net VEXT
Other:
- board text added: "1.5k"
- board text added: "17"
- board text added: "18"
- board text added: "23"
- board text added: "24"
- board text added: "25"
- board text added: "33"
- board text added: "4.952MHz"
- board text added: "C"
- board text added: "CE0"
- board text added: "CE1"
- board text added: "DC"
- board text added: "DD"
- board text added: "DRV8838"
- board text added: "P2_0"
- board text added: "R"
- board text added: "T3_P0"
- board text added: "T3_P1"
- board text added: "nSLEEP"
- board text removed: "1"
- board text removed: "100k"
- board text removed: "2"
- board text removed: "3"
- board text removed: "4.7k"
- board text removed: "4.9512MHz"
- board text removed: "4x 100k"
- board text removed: "ADS1243"
- board text removed: "BLE112A"
- board text removed: "C0"
- board text removed: "C1"
- board text removed: "C2"
- board text removed: "C3"
- board text removed: "C4"
- board text removed: "C5"
- board text removed: "C6"
- board text removed: "C7"
- board text removed: "CC_DEBUG"
- board text removed: "DRDY"
- board text removed: "INT1"
- board text removed: "INT2"
- board text removed: "MMA8451"
- board text removed: "P0_6"
- board text removed: "P0_7"
- board text removed: "P1_1"
- board text removed: "PCT2075"
- board text removed: "PDWN"
- board text removed: "R0"
- board text removed: "R1"
- board text removed: "R2"
- board text removed: "R3"
- board text removed: "R4"
- board text removed: "R5"
- board text removed: "R6"
- board text removed: "R7"
- board text removed: "SD1206S040S2R0"
- board text removed: "TXB0104"
- board text removed: "VBATT"
- board text removed: "VEXT"
