File: hardware/main.sch (EAGLE design)
At the start: 58 parts

Commit message: Hardware revision 2, as ordered.
Parts:
- removed R9: 100k, rcl:R-US_R0603
- removed SERVO1, SERVO2, SERVO3, SERVO4: HDR_1X3, bleHAT:HDR_1X3
- removed U$8: TXB0104, bleHAT:TXB0104
- added 3V3_PI, CS0, CS1, CS2, CS3, CS4, CS5, R16, R17, R8, R_DRDY, R_INT1, R_INT2, R_SCL, R_SDA: (no value), rcl:R-US_R0603
- added C18, C19, C20, C21, C22, C8: (no value), resistor:C-EUC0603
- added JP6: (no value), bleHAT:PINHD-1X6
- added PWM1, PWM2, PWM3, PWM4: HDR_1X3, bleHAT:HDR_1X3
- added R22, R23, R24, R25, R30, R31: (no value), resistor:R-US_R1206
- added U$5, U$7: DRV8838, bleHAT:DRV8838
- JP2: device bleHAT:PINHD-1X7 -> bleHAT:PINHD-1X5
- JP3: device bleHAT:PINHD-1X5 -> bleHAT:PINHD-1X6
- JP4: device bleHAT:PINHD-1X3 -> bleHAT:PINHD-1X2
- JP5: device pinhead:PINHD-1X1 -> bleHAT:PINHD-1X2
Connections:
- removed net N$36: R9.1, U$8.OE
- removed net PDWN_N: BLE112A.P1_3, JP3.1, U$3.PDWN_N
- removed net PWM1_5V0: SERVO4.2, U$8.B4
- removed net PWM2_5V0: SERVO3.2, U$8.B3
- removed net PWM3_5V0: SERVO2.2, U$8.B2
- removed net PWM4_5V0: SERVO1.2, U$8.B1
- new net 3V3_PI: 3V3_PI.1, C11.2, PCT2075.VCC, R14.2, R15.2, U$4.SA0, U$4.VDD, U$4.VDDIO
- new net 3V3_PI_BYP: 3V3_PI.2, JP1.1
- new net GPIO17_PI: JP1.11, R_INT2.2
- new net GPIO18_PI: JP1.12, R_DRDY.1
- new net GPIO4_PI: JP1.7, R_INT1.2
- new net I2C_SCL_PI: JP1.5, R_SCL.2
- new net I2C_SDA_PI: JP1.3, R_SDA.2
- new net N$12: JP4.1, U$5.OUT2
- new net N$13: CS2.2, PWM2.3, R22.1
- new net N$14: CS3.1, PWM1.3, R23.1
- new net N$15: CS0.2, PWM4.3, R25.2
- new net N$16: CS1.1, PWM3.3, R24.2
- new net N$21: JP4.2, U$5.OUT1
- new net N$22: JP5.1, U$7.OUT2
- new net N$23: JP5.2, U$7.OUT1
- new net N$26: CS4.1, R30.2, U$5.GND
- new net N$27: CS5.1, R31.2, U$7.GND
- new net P1_0: BLE112A.P1_0, JP3.4, R17.1
- new net P2_0: BLE112A.P2_0, JP2.3
- new net SLEEP_N: BLE112A.P1_3, JP3.1, U$3.PDWN_N, U$5.NSL, U$7.NSL
- new net TMR3_PWM0: BLE112A.P1_6, JP2.5, U$7.EN
- new net TMR3_PWM1: BLE112A.P1_7, JP2.4, U$5.EN
- new net USB+: BLE112A.USB+, R17.2, R8.2
- new net USB-: BLE112A.USB-, R16.2
- net 3V3: now also U$5.VCC, U$7.VCC; no longer C11.2, PCT2075.VCC, R14.2, R15.2, R9.2, U$4.SA0, U$4.VDD, U$4.VDDIO, U$8.VA
- net 5V0: now also C18.2, C19.2, C20.2, C21.2, C22.2, C8.2, PWM1.2, PWM2.2, PWM3.2, PWM4.2, U$5.VM, U$7.VM; no longer SERVO1.1, SERVO2.1, SERVO3.1, SERVO4.1, U$8.VB
- net AIN0: now also CS4.2
- net AIN1: now also CS5.2
- net AIN4: now also CS3.2
- net AIN5: now also CS2.1
- net AIN6: now also CS0.1
- net AIN7: now also CS1.2
- net ANALOG0: now also JP6.1; no longer JP2.7
- net ANALOG1: now also JP6.2; no longer JP2.6
- net DC: now also JP2.1, U$7.PH
- net DD: now also JP2.2, U$5.PH
- net DRDY_N: now also R_DRDY.2; no longer BLE112A.P1_2, JP2.1
- net GND: now also C18.1, C19.1, C20.1, C21.1, C22.1, C8.1, R22.2, R23.2, R24.1, R25.1, R30.1, R31.1; no longer SERVO1.3, SERVO2.3, SERVO3.3, SERVO4.3, U$8.GND
- net INT1: now also R_INT1.1; no longer JP5.1
- net INT2: now also R_INT2.1; no longer BLE112A.P2_0, JP4.1
- net N$3: now also R8.1; no longer BLE112A.USB+
- net N$4: now also R16.1; no longer BLE112A.USB-
- net PWM1: now also BLE112A.P1_2, PWM1.1; no longer BLE112A.P1_1, U$8.A4
- net PWM2: now also BLE112A.P1_1, PWM2.1; no longer BLE112A.P1_0, U$8.A3
- net PWM3: now also JP3.5, PWM3.1; no longer JP3.4, U$8.A2
- net PWM4: now also JP3.6, PWM4.1; no longer JP3.5, U$8.A1
- net SCL: now also R_SCL.1; no longer BLE112A.P1_7, JP4.2
- net SDA: now also R_SDA.1; no longer BLE112A.P1_6, JP4.3
- net SPI_CLK: now also JP6.4; no longer JP2.4
- net SPI_MISO: now also JP6.6; no longer JP2.2
- net SPI_MOSI: now also JP6.5; no longer JP2.3
- net SPI_SS: now also JP6.3; no longer JP2.5
Other:
- moved on the sheet: C14, JP1
